File: Quad Joystick Mixer/audioInput.kicad_sch (KiCad schematic)
At the start: 19 parts, among them J2 NMJ6HCD, J3 NMJ6HCD, U4 OPA1692xD

Commit message: a few notes about changes
Other:
- note added: "todo: add zener to keep signal +/- 2.5V"
Changed lines of the file:
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@@
+    (stroke (width 0) (type default))
+  )
+  (wire (pts (xy 100.33 73.025) (xy 102.87 73.025))
     (stroke (width 0) (type default))
   )
   (wire (pts (xy 154.94 75.565) (xy 169.545 75.565))
-    (stroke (width 0) (type default))
-  )
-  (wire (pts (xy 100.33 73.025) (xy 102.87 73.025))
     (stroke (width 0) (type default))
   )
@@
     (stroke (width 0) (type default))
   )
-  (wire (pts (xy 169.545 75.565) (xy 172.085 75.565))
+  (wire (pts (xy 169.545 75.565) (xy 178.435 75.565))
     (stroke (width 0) (type default))
   )
@@
     (effects (font (size 1.27 1.27)) (justify left bottom))
   )
+  (text "todo: add zener to keep signal +/- 2.5V" (at 156.845 80.645 0)
+    (effects (font (size 1.27 1.27)) (justify left bottom))
+  )
   (hierarchical_label "Channel2_Input" (shape output) (at 172.085 127.635 0) (fields_autoplaced)
     (effects (font (size 1.27 1.27)) (justify left))
   )
-  (hierarchical_label "Channel1_Input" (shape output) (at 172.085 75.565 0) (fields_autoplaced)
+  (hierarchical_label "Channel1_Input" (shape output) (at 178.435 75.565 0) (fields_autoplaced)
     (effects (font (size 1.27 1.27)) (justify left))
   )

Commit message: more progress on schematic
Parts:
- added D12, D13, D14, D15: MMSZ5222BT1G, Diode_SMD:D_SOD-123, symbol Device:D_Zener
Connections:
- net Channel1_Input: now also D12.2 (A)
- net Channel2_Input: now also D14.2 (A)
- net GND: now also D13.2 (A), D15.2 (A)
- new net: D12.1 (K), D13.1 (K)
- new net: D14.1 (K), D15.1 (K)
Other:
- note removed: "todo: add zener to keep signal +/- 2.5V"
Changed lines of the file:
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@@
   (junction (at 135.255 64.77) (diameter 0) (color 0 0 0 0)
   )
+  (junction (at 174.625 75.565) (diameter 0) (color 0 0 0 0)
+  )
   (junction (at 100.33 137.795) (diameter 0) (color 0 0 0 0)
   )
@@
   )
   (junction (at 217.805 107.95) (diameter 0) (color 0 0 0 0)
+  )
+  (junction (at 163.83 127.635) (diameter 0) (color 0 0 0 0)
   )
   (no_connect (at 96.52 132.715))
@@
     (stroke (width 0) (type default))
   )
+  (wire (pts (xy 174.625 96.52) (xy 174.625 98.425))
+    (stroke (width 0) (type default))
+  )
   (wire (pts (xy 132.08 78.105) (xy 132.08 81.28))
     (stroke (width 0) (type default))
@@
     (stroke (width 0) (type default))
   )
+  (wire (pts (xy 163.83 147.32) (xy 163.83 149.225))
+    (stroke (width 0) (type default))
+  )
   (wire (pts (xy 96.52 125.095) (xy 100.33 125.095))
     (stroke (width 0) (type default))
@@
     (stroke (width 0) (type default))
   )
+  (wire (pts (xy 174.625 75.565) (xy 174.625 79.375))
+    (stroke (width 0) (type default))
+  )
   (wire (pts (xy 100.33 73.025) (xy 102.87 73.025))
     (stroke (width 0) (type default))
@@
     (stroke (width 0) (type default))
   )
+  (wire (pts (xy 163.83 137.795) (xy 163.83 139.7))
+    (stroke (width 0) (type default))
+  )
   (wire (pts (xy 148.59 52.705) (xy 135.255 52.705))
     (stroke (width 0) (type default))
@@
     (stroke (width 0) (type default))
   )
+  (wire (pts (xy 174.625 86.995) (xy 174.625 88.9))
+    (stroke (width 0) (type default))
+  )
   (wire (pts (xy 100.33 75.565) (xy 100.33 73.025))
     (stroke (width 0) (type default))
@@
     (stroke (width 0) (type default))
   )
-  (wire (pts (xy 154.94 127.635) (xy 169.545 127.635))
+  (wire (pts (xy 154.94 127.635) (xy 163.83 127.635))
+    (stroke (width 0) (type default))
+  )
+  (wire (pts (xy 163.83 127.635) (xy 169.545 127.635))
     (stroke (width 0) (type default))
   )
@@
     (stroke (width 0) (type default))
   )
-  (wire (pts (xy 169.545 75.565) (xy 178.435 75.565))
+  (wire (pts (xy 169.545 75.565) (xy 174.625 75.565))
     (stroke (width 0) (type default))
   )
@@
     (stroke (width 0) (type default))
   )
+  (wire (pts (xy 174.625 75.565) (xy 178.435 75.565))
+    (stroke (width 0) (type default))
+  )
   (wire (pts (xy 161.925 111.76) (xy 161.925 116.84))
     (stroke (width 0) (type default))
@@
   )
   (wire (pts (xy 156.21 60.96) (xy 156.21 59.69))
+    (stroke (width 0) (type default))
+  )
+  (wire (pts (xy 163.83 127.635) (xy 163.83 130.175))
     (stroke (width 0) (type default))
   )
@@
   )
   (text "Gain control -20dB (0.1x) -> 40dB (100x)" (at 87.63 113.665 0)
-    (effects (font (size 1.27 1.27)) (justify left bottom))
-  )
-  (text "todo: add zener to keep signal +/- 2.5V" (at 156.845 80.645 0)
     (effects (font (size 1.27 1.27)) (justify left bottom))
   )
@@
     )
   )
+  (symbol (lib_id "Device:D_Zener") (at 174.625 92.71 270) (unit 1)
+    (in_bom yes) (on_board yes) (dnp no) (fields_autoplaced)
+    (property "Reference" "D13" (at 177.8 91.44 90)
+      (effects (font (size 1.27 1.27)) (justify left))
+    )
+    (property "Value" "MMSZ5222BT1G" (at 177.8 93.98 90)
+      (effects (font (size 1.27 1.27)) (justify left))
+    )
+    (property "Footprint" "Diode_SMD:D_SOD-123" (at 174.625 92.71 0)
+      (effects (font (size 1.27 1.27)) hide)
+    )
+    (property "Datasheet" "~" (at 174.625 92.71 0)
+      (effects (font (size 1.27 1.27)) hide)
+    )
+    (pin "1")
+    (pin "2")
+    (instances
+      (project "Quad Joystick Mixer"
+        (path "/e9da4955-68c1-4335-ab8e-8a9cc0328d2d/fc10d8f3-a65b-4c3f-8991-d4833c1f4146"
+          (reference "D13") (unit 1)
+        )
+      )
+    )
+  )
   (symbol (lib_id "Device:C") (at 152.4 104.775 90) (unit 1)
     (in_bom yes) (on_board yes) (dnp no) (fields_autoplaced)
@@
     )
   )
+  (symbol (lib_id "Device:D_Zener") (at 163.83 133.985 90) (unit 1)
+    (in_bom yes) (on_board yes) (dnp no) (fields_autoplaced)
+    (property "Reference" "D14" (at 167.005 132.715 90)
+      (effects (font (size 1.27 1.27)) (justify right))
+    )
+    (property "Value" "MMSZ5222BT1G" (at 167.005 135.255 90)
+      (effects (font (size 1.27 1.27)) (justify right))
+    )
+    (property "Footprint" "Diode_SMD:D_SOD-123" (at 163.83 133.985 0)
+      (effects (font (size 1.27 1.27)) hide)
+    )
+    (property "Datasheet" "~" (at 163.83 133.985 0)
+      (effects (font (size 1.27 1.27)) hide)
+    )
+    (pin "1")
+    (pin "2")
+    (instances
+      (project "Quad Joystick Mixer"
+        (path "/e9da4955-68c1-4335-ab8e-8a9cc0328d2d/fc10d8f3-a65b-4c3f-8991-d4833c1f4146"
+          (reference "D14") (unit 1)
+        )
+      )
+    )
+  )
   (symbol (lib_id "Device:R_US") (at 142.875 64.77 90) (unit 1)
     (in_bom yes) (on_board yes) (dnp no) (fields_autoplaced)
@@
         (path "/e9da4955-68c1-4335-ab8e-8a9cc0328d2d/fc10d8f3-a65b-4c3f-8991-d4833c1f4146"
           (reference "RV2") (unit 1)
+        )
+      )
+    )
+  )
+  (symbol (lib_id "Device:D_Zener") (at 174.625 83.185 90) (unit 1)
+    (in_bom yes) (on_board yes) (dnp no) (fields_autoplaced)
+    (property "Reference" "D12" (at 177.8 81.915 90)
+      (effects (font (size 1.27 1.27)) (justify right))
+    )
+    (property "Value" "MMSZ5222BT1G" (at 177.8 84.455 90)
+      (effects (font (size 1.27 1.27)) (justify right))
+    )
+    (property "Footprint" "Diode_SMD:D_SOD-123" (at 174.625 83.185 0)
+      (effects (font (size 1.27 1.27)) hide)
+    )
+    (property "Datasheet" "~" (at 174.625 83.185 0)
+      (effects (font (size 1.27 1.27)) hide)
+    )
+    (pin "1")
+    (pin "2")
+    (instances
+      (project "Quad Joystick Mixer"
+        (path "/e9da4955-68c1-4335-ab8e-8a9cc0328d2d/fc10d8f3-a65b-4c3f-8991-d4833c1f4146"
+          (reference "D12") (unit 1)
         )
       )
@@
         (path "/e9da4955-68c1-4335-ab8e-8a9cc0328d2d/fc10d8f3-a65b-4c3f-8991-d4833c1f4146"
           (reference "R15") (unit 1)
+        )
+      )
+    )
+  )
+  (symbol (lib_id "Device:D_Zener") (at 163.83 143.51 270) (unit 1)
+    (in_bom yes) (on_board yes) (dnp no) (fields_autoplaced)
+    (property "Reference" "D15" (at 167.005 142.24 90)
+      (effects (font (size 1.27 1.27)) (justify left))
+    )
+    (property "Value" "MMSZ5222BT1G" (at 167.005 144.78 90)
+      (effects (font (size 1.27 1.27)) (justify left))
+    )
+    (property "Footprint" "Diode_SMD:D_SOD-123" (at 163.83 143.51 0)
+      (effects (font (size 1.27 1.27)) hide)
+    )
+    (property "Datasheet" "~" (at 163.83 143.51 0)
+      (effects (font (size 1.27 1.27)) hide)
+    )
+    (pin "1")
+    (pin "2")
+    (instances
+      (project "Quad Joystick Mixer"
+        (path "/e9da4955-68c1-4335-ab8e-8a9cc0328d2d/fc10d8f3-a65b-4c3f-8991-d4833c1f4146"
+          (reference "D15") (unit 1)
+        )
+      )
+    )
+  )
+  (symbol (lib_id "power:GND") (at 174.625 98.425 0) (unit 1)
+    (in_bom yes) (on_board yes) (dnp no) (fields_autoplaced)
+    (property "Reference" "#PWR016" (at 174.625 104.775 0)
+      (effects (font (size 1.27 1.27)) hide)
+    )
+    (property "Value" "GND" (at 174.625 103.505 0)
+      (effects (font (size 1.27 1.27)) hide)
+    )
+    (property "Footprint" "" (at 174.625 98.425 0)
+      (effects (font (size 1.27 1.27)) hide)
+    )
+    (property "Datasheet" "" (at 174.625 98.425 0)
+      (effects (font (size 1.27 1.27)) hide)
+    )
+    (pin "1")
+    (instances
+      (project "Quad Joystick Mixer"
+        (path "/e9da4955-68c1-4335-ab8e-8a9cc0328d2d/fc10d8f3-a65b-4c3f-8991-d4833c1f4146"
+          (reference "#PWR016") (unit 1)
         )
       )
@@
         )
       )
+    )
+  )
+  (symbol (lib_id "power:GND") (at 163.83 149.225 0) (unit 1)
+    (in_bom yes) (on_board yes) (dnp no) (fields_autoplaced)
+    (property "Reference" "#PWR020" (at 163.83 155.575 0)
+      (effects (font (size 1.27 1.27)) hide)
+    )
+    (property "Value" "GND" (at 163.83 154.305 0)
+      (effects (font (size 1.27 1.27)) hide)
+    )
+    (property "Footprint" "" (at 163.83 149.225 0)
+      (effects (font (size 1.27 1.27)) hide)
+    )
+    (property "Datasheet" "" (at 163.83 149.225 0)
+      (effects (font (size 1.27 1.27)) hide)
+    )
+    (pin "1")
+    (instances
+      (project "Quad Joystick Mixer"
+        (path "/e9da4955-68c1-4335-ab8e-8a9cc0328d2d/fc10d8f3-a65b-4c3f-8991-d4833c1f4146"
+          (reference "#PWR020") (unit 1)
+        )
+      )

Commit message: finished first draft of the schematic
Other:
- note added: "Two Channels of Audio Input"
- title: (none) -> Quadrophonic Joystick Mixer
- moved on the sheet: C12, C13, C2, D12, D13, D14, D15, J2, J3, R14, R15, R16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

Commit message: ok the draft wasn't done but now i think it is
Parts:
- added TP1 (x2): TestPoint, TestPoint:TestPoint_THTPad_D1.5mm_Drill0.7mm, symbol Connector:TestPoint
Connections:
- net Channel1_Input: now also TP1.1
- net Channel2_Input: now also TP1.1
Changed lines of the file:
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@@
   (junction (at 171.45 157.48) (diameter 0) (color 0 0 0 0)
   )
+  (junction (at 228.6 160.02) (diameter 0) (color 0 0 0 0)
+  )
   (junction (at 219.71 149.225) (diameter 0) (color 0 0 0 0)
   )
@@
   )
   (junction (at 227.33 149.225) (diameter 0) (color 0 0 0 0)
+  )
+  (junction (at 234.95 107.95) (diameter 0) (color 0 0 0 0)
   )
   (junction (at 193.04 105.41) (diameter 0) (color 0 0 0 0)
@@
   (no_connect (at 154.305 162.56))
   (no_connect (at 154.305 110.49))
+  (wire (pts (xy 234.95 104.14) (xy 234.95 107.95))
+    (stroke (width 0) (type default))
+  )
   (wire (pts (xy 158.115 118.11) (xy 158.115 121.285))
     (stroke (width 0) (type default))
@@
     (stroke (width 0) (type default))
   )
+  (wire (pts (xy 234.95 107.95) (xy 236.22 107.95))
+    (stroke (width 0) (type default))
+  )
   (wire (pts (xy 154.305 160.02) (xy 158.115 160.02))
     (stroke (width 0) (type default))
@@
     (stroke (width 0) (type default))
   )
+  (wire (pts (xy 228.6 156.845) (xy 228.6 160.02))
+    (stroke (width 0) (type default))
+  )
   (wire (pts (xy 227.33 97.155) (xy 219.71 97.155))
     (stroke (width 0) (type default))
@@
     (stroke (width 0) (type default))
   )
+  (wire (pts (xy 236.22 104.14) (xy 234.95 104.14))
+    (stroke (width 0) (type default))
+  )
   (wire (pts (xy 171.45 161.29) (xy 171.45 157.48))
     (stroke (width 0) (type default))
@@
     (stroke (width 0) (type default))
   )
-  (wire (pts (xy 227.33 160.02) (xy 229.87 160.02))
+  (wire (pts (xy 227.33 160.02) (xy 228.6 160.02))
     (stroke (width 0) (type default))
   )
@@
     (stroke (width 0) (type default))
   )
-  (wire (pts (xy 232.41 107.95) (xy 236.22 107.95))
+  (wire (pts (xy 232.41 107.95) (xy 234.95 107.95))
     (stroke (width 0) (type default))
   )
@@
     (stroke (width 0) (type default))
   )
+  (wire (pts (xy 228.6 160.02) (xy 229.87 160.02))
+    (stroke (width 0) (type default))
+  )
   (wire (pts (xy 171.45 157.48) (xy 180.34 157.48))
     (stroke (width 0) (type default))
@@
   )
   (wire (pts (xy 189.865 121.285) (xy 189.865 123.825))
+    (stroke (width 0) (type default))
+  )
+  (wire (pts (xy 229.87 156.845) (xy 228.6 156.845))
     (stroke (width 0) (type default))
   )
@@
     )
   )
+  (symbol (lib_id "Connector:TestPoint") (at 236.22 104.14 270) (unit 1)
+    (in_bom yes) (on_board yes) (dnp no) (fields_autoplaced)
+    (property "Reference" "TP1" (at 241.935 104.14 90)
+      (effects (font (size 1.27 1.27)) (justify left))
+    )
+    (property "Value" "TestPoint" (at 238.252 106.045 0)
+      (effects (font (size 1.27 1.27)) (justify left) hide)
+    )
+    (property "Footprint" "TestPoint:TestPoint_THTPad_D1.5mm_Drill0.7mm" (at 236.22 109.22 0)
+      (effects (font (size 1.27 1.27)) hide)
+    )
+    (property "Datasheet" "~" (at 236.22 109.22 0)
+      (effects (font (size 1.27 1.27)) hide)
+    )
+    (pin "1")
+    (instances
+      (project "Quad Joystick Mixer"
+        (path "/e9da4955-68c1-4335-ab8e-8a9cc0328d2d/70e873e8-c2f7-42de-91d7-3f147d0d972e"
+          (reference "TP1") (unit 1)
+        )
+        (path "/e9da4955-68c1-4335-ab8e-8a9cc0328d2d/fc10d8f3-a65b-4c3f-8991-d4833c1f4146"
+          (reference "TP6") (unit 1)
+        )
+      )
+    )
+  )
   (symbol (lib_id "Device:R_US") (at 200.66 149.225 90) (unit 1)
     (in_bom yes) (on_board yes) (dnp no) (fields_autoplaced)
@@
         )
       )
+    )
+  )
+  (symbol (lib_id "Connector:TestPoint") (at 229.87 156.845 270) (unit 1)
+    (in_bom yes) (on_board yes) (dnp no) (fields_autoplaced)
+    (property "Reference" "TP1" (at 235.585 156.845 90)
+      (effects (font (size 1.27 1.27)) (justify left))
+    )
+    (property "Value" "TestPoint" (at 231.902 158.75 0)
+      (effects (font (size 1.27 1.27)) (justify left) hide)
+    )
+    (property "Footprint" "TestPoint:TestPoint_THTPad_D1.5mm_Drill0.7mm" (at 229.87 161.925 0)
+      (effects (font (size 1.27 1.27)) hide)
+    )
+    (property "Datasheet" "~" (at 229.87 161.925 0)
+      (effects (font (size 1.27 1.27)) hide)
+    )
+    (pin "1")
+    (instances
+      (project "Quad Joystick Mixer"
+        (path "/e9da4955-68c1-4335-ab8e-8a9cc0328d2d/70e873e8-c2f7-42de-91d7-3f147d0d972e"
+          (reference "TP1") (unit 1)
+        )
+        (path "/e9da4955-68c1-4335-ab8e-8a9cc0328d2d/fc10d8f3-a65b-4c3f-8991-d4833c1f4146"
+          (reference "TP7") (unit 1)
+        )
+      )

Commit message: clean up after review, working through BOM
Parts:
- C2: value 22pF -> 10pF; DK PN 1276-1029-1-ND -> 399-C0805C100J5GAC7800CT-ND; MPN CL21B105KBFNNNE -> C0805C100J5GAC7800
- D12, D13, D14, D15: DK PN (none) -> MMSZ5222BT1GOSCT-ND; MPN (none) -> MMSZ5222BT1G
Changed lines of the file:
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@@
+      (effects (font (size 1.27 1.27)) hide)
+    )
+    (property "DK PN" "MMSZ5222BT1GOSCT-ND" (at 232.41 125.095 0)
+      (effects (font (size 1.27 1.27)) hide)
+    )
+    (property "MPN" "MMSZ5222BT1G" (at 232.41 125.095 0)
       (effects (font (size 1.27 1.27)) hide)
     )
@@
       (effects (font (size 1.27 1.27)))
     )
-    (property "Value" "22pF" (at 210.185 132.715 90)
+    (property "Value" "10pF" (at 210.185 132.715 90)
       (effects (font (size 1.27 1.27)))
     )
@@
       (effects (font (size 1.27 1.27)) hide)
     )
-    (property "DK PN" "1276-1029-1-ND" (at 210.185 137.16 0)
-      (effects (font (size 1.27 1.27)) hide)
-    )
-    (property "MPN" "CL21B105KBFNNNE" (at 210.185 137.16 0)
+    (property "DK PN" "399-C0805C100J5GAC7800CT-ND" (at 210.185 137.16 0)
+      (effects (font (size 1.27 1.27)) hide)
+    )
+    (property "MPN" "C0805C100J5GAC7800" (at 210.185 137.16 0)
       (effects (font (size 1.27 1.27)) hide)
     )
@@
       (effects (font (size 1.27 1.27)) hide)
     )
+    (property "DK PN" "MMSZ5222BT1GOSCT-ND" (at 221.615 166.37 0)
+      (effects (font (size 1.27 1.27)) hide)
+    )
+    (property "MPN" "MMSZ5222BT1G" (at 221.615 166.37 0)
+      (effects (font (size 1.27 1.27)) hide)
+    )
     (pin "1")
     (pin "2")
@@
       (effects (font (size 1.27 1.27)) hide)
     )
+    (property "DK PN" "MMSZ5222BT1GOSCT-ND" (at 232.41 115.57 0)
+      (effects (font (size 1.27 1.27)) hide)
+    )
+    (property "MPN" "MMSZ5222BT1G" (at 232.41 115.57 0)
+      (effects (font (size 1.27 1.27)) hide)
+    )
     (pin "1")
     (pin "2")
@@
     )
     (property "Datasheet" "~" (at 221.615 175.895 0)
+      (effects (font (size 1.27 1.27)) hide)
+    )
+    (property "DK PN" "MMSZ5222BT1GOSCT-ND" (at 221.615 175.895 0)
+      (effects (font (size 1.27 1.27)) hide)
+    )
+    (property "MPN" "MMSZ5222BT1G" (at 221.615 175.895 0)
       (effects (font (size 1.27 1.27)) hide)
     )
@@
       (effects (font (size 1.27 1.27)))
     )
-    (property "Value" "22pF" (at 210.185 80.645 90)
+    (property "Value" "10pF" (at 210.185 80.645 90)
       (effects (font (size 1.27 1.27)))
     )
@@
       (effects (font (size 1.27 1.27)) hide)
     )
-    (property "DK PN" "1276-1029-1-ND" (at 210.185 85.09 0)
-      (effects (font (size 1.27 1.27)) hide)
-    )
-    (property "MPN" "CL21B105KBFNNNE" (at 210.185 85.09 0)
-      (effects (font (size 1.27 1.27)) hide)
-    )
+    (property "DK PN" "399-C0805C100J5GAC7800CT-ND" (at 210.185 85.09 0)
+      (effects (font (size 1.27 1.27)) hide)
+    )
+    (property "MPN" "C0805C100J5GAC7800" (at 210.185 85.09 0)
+      (effects (font (size 1.27 1.27)) hide)
+    )

Commit message: finish adding parts to the BOM
Parts:
- C12, C13, C2, D12, D13, D14, D15: Source (none) -> DK
- J2, J3: Source (none) -> SBP
- R14, R19: footprint (none) -> Resistor_SMD:R_0805_2012Metric_Pad1.20x1.40mm_HandSolder; DK PN (none) -> RMCF0805FT100KCT-ND; MPN (none) -> RMCF0805FT100K; Source (none) -> DK
- R15, R18: value 5k -> 4.7k; footprint (none) -> Resistor_SMD:R_0805_2012Metric_Pad1.20x1.40mm_HandSolder; DK PN (none) -> RMCF0805JT4K70CT-ND; MPN (none) -> RMCF0805JT4K70; Source (none) -> DK
- R16, R17: value 500 -> 470; footprint (none) -> Resistor_SMD:R_0805_2012Metric_Pad1.20x1.40mm_HandSolder; DK PN (none) -> RMCF0805FT470RCT-ND; MPN (none) -> RMCF0805FT470R; Source (none) -> DK
- RV1, RV2: footprint (none) -> Eyewool Pots:StomboxParts_9MM; Source (none) -> SBP
- TP1: Source (none) -> NA
- U4: value OPA1692xD -> TL072; DK PN (none) -> 296-TL072HIDRCT-ND; MPN (none) -> TL072HIDR; Source (none) -> DK
