File: Quad Joystick Mixer/digitalPot.kicad_sch (KiCad schematic)
At the start: 40 parts, among them U4 TL072, U8 DS1881Z-050+, U9 DS1881Z-050+

Commit message: work on placement and layout
Parts:
- D16: footprint BZT52C4V7-13-F -> Diode_SMD:D_SOD-123
Changed lines of the file:
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@@
         )
         (path "/e9da4955-68c1-4335-ab8e-8a9cc0328d2d/6b806f6d-da33-48ec-b81c-6968195ad9ad"
-          (reference "U14") (unit 1)
+          (reference "U15") (unit 1)
         )
       )
@@
         )
         (path "/e9da4955-68c1-4335-ab8e-8a9cc0328d2d/6b806f6d-da33-48ec-b81c-6968195ad9ad"
-          (reference "U18") (unit 3)
+          (reference "U16") (unit 3)
         )
       )
@@
         )
         (path "/e9da4955-68c1-4335-ab8e-8a9cc0328d2d/6b806f6d-da33-48ec-b81c-6968195ad9ad"
-          (reference "U16") (unit 3)
+          (reference "U14") (unit 3)
         )
       )
@@
         )
         (path "/e9da4955-68c1-4335-ab8e-8a9cc0328d2d/6b806f6d-da33-48ec-b81c-6968195ad9ad"
-          (reference "U18") (unit 3)
+          (reference "U15") (unit 3)
         )
       )
@@
       (effects (font (size 1.27 1.27)) (justify left))
     )
-    (property "Footprint" "BZT52C4V7-13-F" (at 133.35 72.39 0)
-      (effects (font (size 1.27 1.27)) hide)
-    )
+    (property "Footprint" "Diode_SMD:D_SOD-123" (at 133.35 72.39 0)
+      (effects (font (size 1.27 1.27)) hide)
+    )

Commit message: major layout progress
Parts:
- removed C13 (x3): 0.1uF, Capacitor_SMD:C_0805_2012Metric_Pad1.18x1.45mm_HandSolder, symbol Device:C
- removed R23, R8: 20k, Resistor_SMD:R_0805_2012Metric_Pad1.20x1.40mm_HandSolder, symbol Device:R_US
- removed U4: TL072, Package_SO:SOIC-8_3.9x4.9mm_P1.27mm, symbol Amplifier_Operational:OPA1692xD
Connections:
- net Earth is gone; now on net GND: C13.2, C13.2, R25.2, R26.2, U8.2 (A2), U8.3 (A1), U8.5 (A0), U9.2 (A2), U9.3 (A1)
- net Mix_Input: no longer names the net of C2.2, D16.1 (K), R14.2, U8.10 (H1), U8.8 (H0), U9.10 (H1), U9.8 (H0)
