File: Quad Joystick Mixer/Quad Joystick Mixer.kicad_pcb (KiCad board)
At the start: 4 copper layers, 215 x 134.8 mm, 253 parts, among them J1 Barrel_Jack_Switch, J2 NMJ6HCD, J3 NMJ6HCD, J4 NMJ6HCD, J5 NMJ6HCD, J6 NMJ6HCD, J7 NMJ6HCD, Q1 2N7002, Q2 2N7002, SW1 SW_DPDT_x2, SW2 Stompbox 1P8T Rotary, SW3 Cherry MX, SW4 Cherry MX, SW5 Cherry MX, SW6 Cherry MX, SW7 Cherry MX, U1 LM338-TO-220, U10 TL072, U11 TL072, U12 TL072, U13 DS1881Z-050+, U14 TL072, U16 TL072, U17 DS1881Z-050+, U19 TL072, U2 LM2990T-12/NOPB, U20 Teensy4.0, U3 AP63200WU, U4 TL072, U5 MCP1755T-5002E/OT, U6 TL072, U7 TL072, U8 DS1881Z-050+, U9 DS1881Z-050+

Commit message: more work no routing the board
Parts:
- moved R40 15.9 mm to (129.0, 112.3)
- turned R20 to -90 degrees
Routing:
- net -12V: track 44.7 -> 48.6 mm, vias 9 -> 11
Changed lines of the file:
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@@
   )
   (footprint "Resistor_SMD:R_2010_5025Metric_Pad1.40x2.65mm_HandSolder" (layer "F.Cu")
-    (at 144.86875 112.31485)
+    (at 129 112.31485)
     (descr "Resistor SMD 2010 (5025 Metric), square (rectangular) end terminal, IPC_7351 nominal with elongated pad for handsoldering. (Body size source: IPC-SM-782 page 72, https://www.pcb-3d.com/wordpress/wp-content/uploads/ipc-sm-782a_amendment_1_and_2.pdf), generated with kicad-footprint-generator")
     (tags "resistor handsolder")
@@
   )
   (footprint "Resistor_SMD:R_2010_5025Metric_Pad1.40x2.65mm_HandSolder" (layer "F.Cu")
-    (at 152.26875 120.48985 90)
+    (at 152.26875 120.48985 -90)
     (descr "Resistor SMD 2010 (5025 Metric), square (rectangular) end terminal, IPC_7351 nominal with elongated pad for handsoldering. (Body size source: IPC-SM-782 page 72, https://www.pcb-3d.com/wordpress/wp-content/uploads/ipc-sm-782a_amendment_1_and_2.pdf), generated with kicad-footprint-generator")
     (tags "resistor handsolder")
@@
     (fp_line (start 2.5 1.25) (end -2.5 1.25)
       (stroke (width 0.1) (type solid)) (layer "F.Fab"))
-    (pad "1" smd roundrect (at -2.4 0 90) (size 1.4 2.65) (layers "F.Cu" "F.Paste" "F.Mask") (roundrect_rratio 0.178571)
+    (pad "1" smd roundrect (at -2.4 0 270) (size 1.4 2.65) (layers "F.Cu" "F.Paste" "F.Mask") (roundrect_rratio 0.178571)
       (net 31 "Net-(U5-VIN)") (pintype "passive"))
-    (pad "2" smd roundrect (at 2.4 0 90) (size 1.4 2.65) (layers "F.Cu" "F.Paste" "F.Mask") (roundrect_rratio 0.178571)
+    (pad "2" smd roundrect (at 2.4 0 270) (size 1.4 2.65) (layers "F.Cu" "F.Paste" "F.Mask") (roundrect_rratio 0.178571)
       (net 4 "+12V") (pintype "passive"))
     (model "${KICAD6_3DMODEL_DIR}/Resistor_SMD.3dshapes/R_2010_5025Metric.wrl"
@@
   (segment (start 142.97625 141.12625) (end 142.97625 139.59375) (width 0.25) (layer "F.Cu") (net 6))
   (segment (start 41.94875 106.06625) (end 41.94875 111.30125) (width 0.762) (layer "F.Cu") (net 6))
+  (segment (start 169.76875 119.05235) (end 171.94765 119.05235) (width 0.254) (layer "F.Cu") (net 6))
   (segment (start 41.77625 100.51125) (end 41.77625 103.01125) (width 0.762) (layer "F.Cu") (net 6))
   (segment (start 206.23875 65.76125) (end 208.16875 65.76125) (width 0.254) (layer "F.Cu") (net 6))
   (segment (start 146.23875 88.28125) (end 148.02125 88.28125) (width 0.254) (layer "F.Cu") (net 6))
   (segment (start 166.41875 66.01125) (end 167.01375 65.41625) (width 0.254) (layer "F.Cu") (net 6))
+  (segment (start 172 119) (end 171.94765 119.05235) (width 0.254) (layer "F.Cu") (net 6))
   (segment (start 204.21375 84.07625) (end 204.23875 84.05125) (width 0.254) (layer "F.Cu") (net 6))
   (segment (start 169.76875 117.01985) (end 169.79375 116.99485) (width 0.254) (layer "F.Cu") (net 6))
@@
   (segment (start 208.16875 65.76125) (end 208.76375 65.16625) (width 0.254) (layer "F.Cu") (net 6))
   (segment (start 213.42625 136.25375) (end 214.01375 135.66625) (width 0.254) (layer "F.Cu") (net 6))
+  (segment (start 213.42625 138.39625) (end 212.60375 138.39625) (width 0.254) (layer "F.Cu") (net 6))
   (segment (start 41.23875 116.01125) (end 41.23875 120.12125) (width 0.762) (layer "F.Cu") (net 6))
   (segment (start 41.94875 106.06625) (end 41.94875 103.18375) (width 0.762) (layer "F.Cu") (net 6))
@@
   (segment (start 228.85125 87.33875) (end 228.85125 85.76875) (width 0.254) (layer "F.Cu") (net 6))
   (segment (start 142.12625 141.12625) (end 141.5 140.5) (width 0.25) (layer "F.Cu") (net 6))
+  (segment (start 212.60375 138.39625) (end 212 139) (width 0.254) (layer "F.Cu") (net 6))
   (via (at 33.48875 103.26125) (size 0.8) (drill 0.4) (layers "F.Cu" "B.Cu") (free) (net 6))
   (via (at 141.5 140.5) (size 0.8) (drill 0.4) (layers "F.Cu" "B.Cu") (net 6))
@@
   (via (at 33.48875 108.975534) (size 0.8) (drill 0.4) (layers "F.Cu" "B.Cu") (free) (net 6))
   (via (at 33.48875 106.118392) (size 0.8) (drill 0.4) (layers "F.Cu" "B.Cu") (free) (net 6))
+  (via (at 171.94765 119.05235) (size 0.8) (drill 0.4) (layers "F.Cu" "B.Cu") (net 6))
   (via (at 33.48875 111.832676) (size 0.8) (drill 0.4) (layers "F.Cu" "B.Cu") (free) (net 6))
   (via (at 33.48875 117.54696) (size 0.8) (drill 0.4) (layers "F.Cu" "B.Cu") (free) (net 6))
   (via (at 33.48875 123.26125) (size 0.8) (drill 0.4) (layers "F.Cu" "B.Cu") (free) (net 6))
+  (via (at 212 139) (size 0.8) (drill 0.4) (layers "F.Cu" "B.Cu") (net 6))
   (segment (start 112.55125 101.19875) (end 112.55125 99.03625) (width 0.508) (layer "F.Cu") (net 7))
   (segment (start 105.98875 107.72375) (end 108.20125 107.72375) (width 0.508) (layer "F.Cu") (net 7))
@@
     (polygon
       (pts
-        (xy 119 106.5)
+        (xy 121 106.5)
         (xy 68.5 106.5)
         (xy 68.5 116)
-        (xy 119 116)
+        (xy 121 116)
       )
     )
@@
     )
   )
+  (zone (net 4) (net_name "+12V") (layer "F.Cu") (hatch edge 0.5)
+    (priority 24)
+    (connect_pads (clearance 0.5))
+    (min_thickness 0.25) (filled_areas_thickness no)
+    (fill yes (thermal_gap 0.5) (thermal_bridge_width 0.5))
+    (polygon
+      (pts
+        (xy 148 121)
+        (xy 156 121)
+        (xy 156 135)
+        (xy 113 135)
+        (xy 113 114)
+        (xy 121 114)
+        (xy 121 127)
+        (xy 148 127)
+      )
+    )
+  )
+  (zone (net 7) (net_name "+5V") (layer "F.Cu") (hatch edge 0.5)
+    (priority 25)
+    (connect_pads (clearance 0.5))
+    (min_thickness 0.25) (filled_areas_thickness no)
+    (fill yes (thermal_gap 0.5) (thermal_bridge_width 0.5))
+    (polygon
+      (pts
+        (xy 123 115)
+        (xy 123 98)
+        (xy 128.5 98)
+        (xy 128.5 115)
+      )
+    )
+  )
   (zone (net 30) (net_name "VCC") (layer "F.Cu") (hatch edge 0.5)
     (priority 4)
@@
     (polygon
       (pts
-        (xy 152.73875 113.51125)
-        (xy 145.23875 113.51125)
-        (xy 145.23875 106.76125)
+        (xy 168.5 117.01125)
+        (xy 130 117.01125)
+        (xy 129.98875 106.76125)
         (xy 152.73875 106.76125)
-        (xy 152.73875 108.01125)
+        (xy 168.5 106.75)
       )
     )
@@
     )
   )
+  (zone (net 6) (net_name "-12V") (layer "In2.Cu") (hatch edge 0.5)
+    (priority 23)
+    (connect_pads (clearance 0.5))
+    (min_thickness 0.25) (filled_areas_thickness no)
+    (fill yes (thermal_gap 0.5) (thermal_bridge_width 0.5))
+    (polygon
+      (pts
+        (xy 174 139)
+        (xy 174 124)
+        (xy 167 124)
+        (xy 167 116)
+        (xy 175 116)
+        (xy 175 121)
+        (xy 181 121)
+        (xy 181 139)
+      )
+    )
+  )
   (zone (net 33) (net_name "+3.3V") (layer "In2.Cu") (hatch edge 0.5)
     (priority 18)
@@
     (polygon
       (pts
-        (xy 152.73875 105.26125)
-        (xy 143.73875 105.26125)
-        (xy 143.73875 96.76125)
-        (xy 155.98875 96.76125)
-        (xy 155.98875 95.76125)
-        (xy 206.23875 95.76125)
-        (xy 206.23875 97.26125)
-        (xy 241.48875 97.26125)
-        (xy 241.48875 92.51125)
-        (xy 211.48875 92.51125)
-        (xy 204.48875 92.51125)
-        (xy 204.48875 92.26125)
-        (xy 137.23875 92.26125)
-        (xy 136.98875 109.26125)
-        (xy 145.23875 109.26125)
-        (xy 145.23875 113.51125)
-        (xy 152.73875 113.51125)
-        (xy 152.73875 112.01125)
+        (xy 151.98875 105.26125)
+        (xy 142.98875 105.26125)
+        (xy 142.98875 96.76125)
+        (xy 155.23875 96.76125)
+        (xy 155.23875 95.76125)
+        (xy 205.48875 95.76125)
+        (xy 205.48875 97.26125)
+        (xy 240.73875 97.26125)
+        (xy 240.73875 92.51125)
+        (xy 210.73875 92.51125)
+        (xy 203.73875 92.51125)
+        (xy 203.73875 92.26125)
+        (xy 136.25 92.26125)
+        (xy 136.23875 109.26125)
+        (xy 129.98875 109.26125)
+        (xy 129.98875 113.51125)
+        (xy 151.98875 113.51125)
+        (xy 151.98875 112.01125)
       )
     )
@@
     (polygon
       (pts
-        (xy 139.5 138.5)
+        (xy 139.5 136.5)
         (xy 139.5 142.5)
         (xy 162.5 142.5)
@@
         (xy 31.5 123)
         (xy 31.5 159)
-        (xy 167.5 159.5)
-        (xy 167.5 138.5)
+        (xy 215.5 159.5)
+        (xy 215.5 136.5)
       )
     )

Commit message: update layout
Parts:
- moved R30 1.28 mm to (141.7, 85.0)
- moved R46 1.28 mm to (139.2, 85.0)
Routing:
- net /Audio Output/B: track 34.8 -> 145.3 mm
- net +12V: track 75.8 -> 90.9 mm, vias 10 -> 17
- net +3.3V: track 166.0 -> 155.9 mm
- net /Audio Input/Channel2_Input: track 133.3 -> 134.9 mm
- net /Audio Output/C: track 148.6 -> 147.3 mm
- net Net-(U16B-+): track 32.5 -> 33.4 mm
- net Net-(C47-Pad2): track 4.96 -> 5.49 mm

Commit message: three nets left to route
Routing:
- net /Audio Output/A: track 34.6 -> 94.3 mm, vias 0 -> 2
- net /Audio Input/Channel1_Input: track 107.2 -> 131.5 mm, vias 0 -> 2
- net /Audio Input/Channel2_Input: track 134.9 -> 154.4 mm, vias 0 -> 2
- net -12V: track 48.1 -> 61.2 mm, vias 11 -> 17
- net Net-(U16A-+): track 31.2 -> 32.0 mm
- net +3.3V: track 155.9 -> 156.7 mm
- net /Audio Output/B: track 145.3 -> 146.0 mm
- added copper zone on B.Cu, net -12V
- added copper zone on B.Cu, net Earth

Commit message: work through DRC errors
Parts:
- added J8: XH-A, Connector_JST:JST_XH_B3B-XH-AM_1x03_P2.50mm_Vertical, F.Cu at (162.5, 156.0)
- added J9: XH-A, Connector_JST:JST_XH_B3B-XH-AM_1x03_P2.50mm_Vertical, F.Cu at (162.5, 148.5)
Routing:
- net Net-(J8-Pin_2): track 9.95 -> 40.0 mm
- net Net-(J9-Pin_2): track 9.57 -> 18.8 mm
- net +3.3V: track 156.7 -> 162.3 mm
- net GND: track 127.8 -> 124.9 mm
- net /Teensy/AB_Control: track 112.9 -> 115.6 mm
- net Earth: track 117.1 -> 115.5 mm
- net /Teensy/CD_Control: track 153.4 -> 154.7 mm
- net /Audio Input/Channel2_Input: track 154.4 -> 153.2 mm
- net +12V: track 90.9 -> 92.0 mm
- net Net-(J4-PadT): track 33.3 -> 32.2 mm
- net Net-(U4A--): track 12.8 -> 11.8 mm
- net -12V: track 61.2 -> 60.4 mm
- net Net-(U10A-+): track 29.8 -> 29.1 mm
- net /SDA0: track 93.8 -> 93.1 mm
- net Net-(U7A-+): track 11.3 -> 10.6 mm
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