File: Quad Joystick Mixer/Quad Joystick Mixer.kicad_pcb (KiCad board)
At the start: 4 copper layers, 215 x 134.8 mm, 255 parts, among them J1 Barrel_Jack_Switch, J2 NMJ6HCD, J3 NMJ6HCD, J4 NMJ6HCD, J5 NMJ6HCD, J6 NMJ6HCD, J7 NMJ6HCD, J8 XH-A, J9 XH-A, Q1 2N7002, Q2 2N7002, SW1 SW_DPDT_x2, SW2 Stompbox 1P8T Rotary, SW3 Cherry MX, SW4 Cherry MX, SW5 Cherry MX, SW6 Cherry MX, SW7 Cherry MX, U1 LM338-TO-220, U10 TL072, U11 TL072, U12 TL072, U13 DS1881Z-050+, U14 TL072, U16 TL072, U17 DS1881Z-050+, U19 TL072, U2 LM2990T-12/NOPB, U20 Teensy4.0, U3 AP63200WU, U4 TL072, U5 MCP1755T-5002E/OT, U6 TL072, U7 TL072, U8 DS1881Z-050+, U9 DS1881Z-050+

Commit message: changed power supply design and everything re routed
Parts:
- removed C14: 100uF, Capacitor_THT:CP_Radial_D8.0mm_P3.50mm
- removed C17, C18: 22uF, Capacitor_SMD:C_1206_3216Metric_Pad1.33x1.80mm_HandSolder
- removed C19, C20, C22: 0.1uF, Capacitor_SMD:C_0805_2012Metric_Pad1.18x1.45mm_HandSolder
- removed C21, C7: 10uF, Capacitor_SMD:C_0805_2012Metric_Pad1.18x1.45mm_HandSolder
- removed C23: 100pF, Capacitor_SMD:C_0805_2012Metric_Pad1.18x1.45mm_HandSolder
- removed D10, D2, D3, D4, D6: B350, Diode_SMD:D_SMA_Handsoldering
- removed D8: LED, LED_THT:LED_D3.0mm_FlatTop
- removed L4: 10uH, Inductor_SMD:L_Abracon_ASPI-0630LR
- removed R1, R2, R6, R7: 0.5R, Resistor_SMD:R_2512_6332Metric_Pad1.40x3.35mm_HandSolder
- removed R10: 3k, Resistor_SMD:R_0805_2012Metric_Pad1.20x1.40mm_HandSolder
- removed R12: 158k, Resistor_SMD:R_0805_2012Metric_Pad1.20x1.40mm_HandSolder
- removed R13: 30k, Resistor_SMD:R_0805_2012Metric_Pad1.20x1.40mm_HandSolder
- removed R4: 270R, Resistor_SMD:R_0805_2012Metric_Pad1.20x1.40mm_HandSolder
- removed R5: 2.32k, Resistor_SMD:R_0805_2012Metric_Pad1.20x1.40mm_HandSolder
- removed SW1: SW_DPDT_x2, Eyewool Switches:Taiway DPDT
- removed U3: AP63200WU, Package_TO_SOT_SMD:TSOT-23-6
- C12, C3, C4: value 2200uF -> 1uF; footprint Capacitor_THT:C_Radial_D16.0mm_H25.0mm_P7.50mm -> Capacitor_SMD:C_0805_2012Metric_Pad1.18x1.45mm_HandSolder
- C13: value 2200uF -> 0.1uF; footprint Capacitor_THT:C_Radial_D16.0mm_H25.0mm_P7.50mm -> Capacitor_SMD:C_0805_2012Metric_Pad1.18x1.45mm_HandSolder
- C5: value 100uF -> 0.1uF; footprint Capacitor_THT:CP_Radial_D8.0mm_P3.50mm -> Capacitor_SMD:C_0805_2012Metric_Pad1.18x1.45mm_HandSolder
- J1: value Barrel_Jack_Switch -> XH-B4B-XH; footprint Eyewool Connectors:Love My Switches 2.1MM PCB Mount DC Jack -> Connector_JST:JST_XH_B4B-XH-AM_1x04_P2.50mm_Vertical
- U1: value LM338-TO-220 -> L78M12ACDT-TR; footprint Package_TO_SOT_THT:TO-220-3_Vertical -> Package_TO_SOT_SMD:TO-252-2
- U2: value LM2990T-12/NOPB -> MC79L12ABDG; footprint Package_TO_SOT_THT:TO-220-3_Vertical -> Package_SO:SOIC-8_3.9x4.9mm_P1.27mm
- moved D5 75.7 mm to (64.8, 39.2), turned to -90 degrees
- moved C82 72.5 mm to (106.8, 102.4)
- moved D22 72.5 mm to (106.8, 105.4)
- moved R82 72.5 mm to (110.3, 101.4)
- moved SW3 72.5 mm to (112.3, 112.5)
- moved TP4 69.8 mm to (85.5, 32.8), turned to 0 degrees
- moved TP2 69.4 mm to (70.0, 53.2)
- moved D7 68.5 mm to (70.0, 58.8)
- moved D1 68.4 mm to (72.5, 42.8)
- moved R9 68.3 mm to (75.5, 58.5), turned to 0 degrees
- moved C2 64.5 mm to (75.5, 53.8)
- moved R11 62.7 mm to (66.5, 62.2)
- moved U1 60.6 mm to (80.1, 49.0)
- moved C1 60.2 mm to (75.5, 56.0)
- moved C15 59.6 mm to (64.5, 46.2)
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Connections:
- C12 pad 1: Earth -> -15V
- C12 pad 2: Net-(C12-Pad2) -> Earth
- C13 pad 1: Earth -> Net-(D5-A)
- C13 pad 2: Net-(C12-Pad2) -> Earth
- C3 pad 1: Net-(C3-Pad1) -> +5V
- C4 pad 1: Net-(C3-Pad1) -> +15V
- D1 pad 2: +12V -> +15V
- D5 pad 1: -12V -> -15V
- J1 pad 1: Earth -> +5V
- J1 pad 2: Net-(SW1A-B) -> Earth
- J1 pad 3: unconnected-(J1-Pad3) -> +15V
- U1 pad 1: Net-(D3-A) -> Net-(D1-K)
- U1 pad 2: +12V -> Earth
- U1 pad 3: Net-(D1-K) -> +12V
- U2 pad 1: Earth -> -12V
- U2 pad 3: -12V -> Net-(D5-A)
- U20 pad 10: /Teensy/Button_3 -> /Teensy/Button_2
- U20 pad 8: /Teensy/Button_1 -> /Teensy/Button_3
- U20 pad 9: /Teensy/Button_2 -> /Teensy/Button_1
Routing:
- net +3.3V: track 162.3 -> 258.4 mm, vias 12 -> 8
- net /Teensy/Button_1: track 134.4 -> 66.3 mm, vias 0 -> 1
- net +5V: track 38.7 -> 88.2 mm
- net /Teensy/Button_2: track 117.2 -> 68.0 mm, vias 0 -> 1
- net Net-(C12-Pad2): track 37.7 -> 0.00 mm
- net Net-(C3-Pad1): track 36.8 -> 0.00 mm
- net Net-(D5-A): track 27.3 -> 0.00 mm
- net -12V: track 60.4 -> 40.7 mm, vias 17 -> 10
- net Net-(D3-A): track 17.5 -> 0.00 mm
- net Net-(SW1A-B): track 15.6 -> 0.00 mm
- net Earth: track 115.5 -> 100.3 mm, vias 56 -> 50
- net Net-(D1-K): track 24.7 -> 9.90 mm
- net VCC: track 36.7 -> 22.1 mm
- net Net-(D2-A): track 14.1 -> 0.00 mm
- net +12V: track 92.0 -> 78.2 mm, vias 17 -> 14
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- added copper zone on F.Cu, net +3.3V
- added copper zone on F.Cu, net Net-(D5-A)
- removed copper zone on F.Cu, net GND
Other:
- board size 215 x 134.8 mm -> 189.3 x 134.8 mm

Commit message: clean up DRC results
Routing:
- net +3.3V: track 258.4 -> 259.3 mm
- net +5V: track 88.2 -> 88.9 mm
- net /Teensy/AB_Control: track 115.6 -> 115.0 mm
