File: Quad Joystick Mixer/Quad Joystick Mixer.kicad_sch (KiCad schematic)
At the start: 0 parts

Commit message: finished first draft of the schematic
Other:
- sheet Joystick renamed User Interface
- sheet Teensy ports: added AB_Control, Button_1, Button_2, Button_3, CD_Control, Channel Selection, LED_1, LED_2, SCL0, SCL1, SCL2, SDA0, SDA1, SDA2; removed none
- sheet User Interface: file joystick.kicad_sch -> userInterface.kicad_sch
- sheet User Interface ports: added Button_1, Button_2, Button_3, Channel Selection, LED_1, LED_2; removed none
- note added: "8x GPIO is replaced with 1x ADC for channel select"
- note added: "Max of 8 digital pots per I2C 2 digital pots per channel 12 channel max for system"

Commit message: ok the draft wasn't done but now i think it is
Parts:
- added R85, R86: DNA, symbol Device:R_US
Connections:
- net Audio Input/Channel1_Input: now also R85.1
- net Audio Input/Channel2_Input: now also R86.1
- net Audio Output/A: now also R85.2
- net Audio Output/D: now also R86.2
Other:
- note added: "R85 and R86 provided for route around debug of audio path as required"
Changed lines of the file:
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@@
     (rev "P1")
   )
+  (junction (at 276.86 71.755) (diameter 0) (color 0 0 0 0)
+  )
   (junction (at 325.755 42.545) (diameter 0) (color 0 0 0 0)
   )
   (junction (at 337.185 53.975) (diameter 0) (color 0 0 0 0)
   )
+  (junction (at 273.685 48.895) (diameter 0) (color 0 0 0 0)
+  )
+  (junction (at 335.28 42.545) (diameter 0) (color 0 0 0 0)
+  )
+  (junction (at 323.215 53.975) (diameter 0) (color 0 0 0 0)
+  )
   (junction (at 333.375 50.165) (diameter 0) (color 0 0 0 0)
   )
@@
     (stroke (width 0) (type default))
   )
+  (wire (pts (xy 297.18 23.495) (xy 273.685 23.495))
+    (stroke (width 0) (type default))
+  )
   (wire (pts (xy 285.75 86.995) (xy 292.1 86.995))
     (stroke (width 0) (type default))
   )
-  (wire (pts (xy 276.86 55.88) (xy 276.86 90.805))
+  (wire (pts (xy 306.07 71.755) (xy 323.215 71.755))
+    (stroke (width 0) (type default))
+  )
+  (wire (pts (xy 276.86 55.88) (xy 276.86 71.755))
     (stroke (width 0) (type default))
   )
@@
     (stroke (width 0) (type default))
   )
-  (wire (pts (xy 325.755 42.545) (xy 356.87 42.545))
+  (wire (pts (xy 273.685 48.895) (xy 291.465 48.895))
+    (stroke (width 0) (type default))
+  )
+  (wire (pts (xy 325.755 42.545) (xy 335.28 42.545))
     (stroke (width 0) (type default))
   )
@@
     (stroke (width 0) (type default))
   )
-  (wire (pts (xy 262.89 48.895) (xy 291.465 48.895))
+  (wire (pts (xy 262.89 48.895) (xy 273.685 48.895))
     (stroke (width 0) (type default))
   )
@@
     (stroke (width 0) (type default))
   )
+  (wire (pts (xy 304.8 23.495) (xy 335.28 23.495))
+    (stroke (width 0) (type default))
+  )
   (wire (pts (xy 170.815 42.545) (xy 174.625 42.545))
     (stroke (width 0) (type default))
@@
     (stroke (width 0) (type default))
   )
+  (wire (pts (xy 323.215 53.975) (xy 337.185 53.975))
+    (stroke (width 0) (type default))
+  )
   (wire (pts (xy 297.18 145.415) (xy 305.435 145.415))
     (stroke (width 0) (type default))
   )
+  (wire (pts (xy 276.86 71.755) (xy 276.86 90.805))
+    (stroke (width 0) (type default))
+  )
   (wire (pts (xy 297.18 142.24) (xy 305.435 142.24))
     (stroke (width 0) (type default))
@@
     (stroke (width 0) (type default))
   )
+  (wire (pts (xy 335.28 42.545) (xy 356.87 42.545))
+    (stroke (width 0) (type default))
+  )
   (wire (pts (xy 262.89 55.88) (xy 276.86 55.88))
     (stroke (width 0) (type default))
@@
     (stroke (width 0) (type default))
   )
+  (wire (pts (xy 323.215 53.975) (xy 323.215 71.755))
+    (stroke (width 0) (type default))
+  )
   (wire (pts (xy 329.565 46.355) (xy 356.87 46.355))
     (stroke (width 0) (type default))
@@
     (stroke (width 0) (type default))
   )
+  (wire (pts (xy 273.685 23.495) (xy 273.685 48.895))
+    (stroke (width 0) (type default))
+  )
   (wire (pts (xy 297.18 155.575) (xy 305.435 155.575))
     (stroke (width 0) (type default))
@@
     (stroke (width 0) (type default))
   )
+  (wire (pts (xy 276.86 71.755) (xy 298.45 71.755))
+    (stroke (width 0) (type default))
+  )
   (wire (pts (xy 337.185 53.975) (xy 356.87 53.975))
     (stroke (width 0) (type default))
   )
-  (wire (pts (xy 320.04 53.975) (xy 337.185 53.975))
+  (wire (pts (xy 320.04 53.975) (xy 323.215 53.975))
+    (stroke (width 0) (type default))
+  )
+  (wire (pts (xy 335.28 23.495) (xy 335.28 42.545))
     (stroke (width 0) (type default))
   )
@@
     (effects (font (size 1.27 1.27)) (justify left bottom))
   )
+  (text "R85 and R86 provided for route around \ndebug of audio path as required"
+    (at 339.0003 29.739 0)
+    (effects (font (size 1.27 1.27)) (justify left bottom))
+  )
   (text "Max of 8 digital pots per I2C\n2 digital pots per channel\n12 channel max for system"
     (at 353.06 144.145 0)
@@
     )
   )
+  (symbol (lib_id "Device:R_US") (at 302.26 71.755 90) (unit 1)
+    (in_bom yes) (on_board yes) (dnp no)
+    (property "Reference" "R86" (at 298.45 69.85 90)
+      (effects (font (size 1.27 1.27)))
+    )
+    (property "Value" "DNA" (at 306.07 69.85 90)
+      (effects (font (size 1.27 1.27)))
+    )
+    (property "Footprint" "" (at 302.514 70.739 90)
+      (effects (font (size 1.27 1.27)) hide)
+    )
+    (property "Datasheet" "~" (at 302.26 71.755 0)
+      (effects (font (size 1.27 1.27)) hide)
+    )
+    (pin "1")
+    (pin "2")
+    (instances
+      (project "Quad Joystick Mixer"
+        (path "/e9da4955-68c1-4335-ab8e-8a9cc0328d2d"
+          (reference "R86") (unit 1)
+        )
+      )
+    )
+  )
   (symbol (lib_id "power:-12V") (at 181.61 39.37 0) (unit 1)
     (in_bom yes) (on_board yes) (dnp no) (fields_autoplaced)
@@
         )
       )
+    )
+  )
+  (symbol (lib_id "Device:R_US") (at 300.99 23.495 90) (unit 1)
+    (in_bom yes) (on_board yes) (dnp no)
+    (property "Reference" "R85" (at 297.18 21.59 90)
+      (effects (font (size 1.27 1.27)))
+    )
+    (property "Value" "DNA" (at 304.8 21.59 90)
+      (effects (font (size 1.27 1.27)))
+    )
+    (property "Footprint" "" (at 301.244 22.479 90)
+      (effects (font (size 1.27 1.27)) hide)
+    )
+    (property "Datasheet" "~" (at 300.99 23.495 0)
+      (effects (font (size 1.27 1.27)) hide)
+    )
+    (pin "1")
+    (pin "2")
+    (instances
+      (project "Quad Joystick Mixer"
+        (path "/e9da4955-68c1-4335-ab8e-8a9cc0328d2d"
+          (reference "R85") (unit 1)
+        )
+      )

Commit message: clean up after review, working through BOM
Parts:
- added NT1: NetTie_2, NetTie:NetTie-2_SMD_Pad2.0mm, symbol Device:NetTie_2
- added R87, R88: DNA, symbol Device:R_US
Connections:
- net Audio Input/Channel1_Input: now also R88.1
- net Audio Input/Channel2_Input: now also R87.1
- net Audio Output/B: now also R88.2
- net Audio Output/C: now also R87.2
- new net Earth: NT1.1
- new net GND: NT1.2
Other:
- note added: "R85 routes input 1 -> A R88 routes input 1 -> B R87 routes input 2 -> C R86 routes input 2 -> D"
- note removed: "R85 and R86 provided for route around debug of audio path as required"
Changed lines of the file:
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@@
   (junction (at 337.185 53.975) (diameter 0) (color 0 0 0 0)
   )
+  (junction (at 341.63 50.165) (diameter 0) (color 0 0 0 0)
+  )
+  (junction (at 277.495 48.895) (diameter 0) (color 0 0 0 0)
+  )
   (junction (at 273.685 48.895) (diameter 0) (color 0 0 0 0)
   )
@@
   (junction (at 323.215 53.975) (diameter 0) (color 0 0 0 0)
   )
+  (junction (at 276.86 66.675) (diameter 0) (color 0 0 0 0)
+  )
+  (junction (at 338.455 46.355) (diameter 0) (color 0 0 0 0)
+  )
   (junction (at 333.375 50.165) (diameter 0) (color 0 0 0 0)
   )
@@
     (stroke (width 0) (type default))
   )
-  (wire (pts (xy 276.86 55.88) (xy 276.86 71.755))
+  (wire (pts (xy 276.86 55.88) (xy 276.86 66.675))
+    (stroke (width 0) (type default))
+  )
+  (wire (pts (xy 341.63 66.675) (xy 341.63 50.165))
     (stroke (width 0) (type default))
   )
@@
     (stroke (width 0) (type default))
   )
-  (wire (pts (xy 273.685 48.895) (xy 291.465 48.895))
+  (wire (pts (xy 273.685 48.895) (xy 277.495 48.895))
+    (stroke (width 0) (type default))
+  )
+  (wire (pts (xy 277.495 29.21) (xy 277.495 48.895))
     (stroke (width 0) (type default))
   )
@@
     (stroke (width 0) (type default))
   )
+  (wire (pts (xy 341.63 50.165) (xy 356.87 50.165))
+    (stroke (width 0) (type default))
+  )
   (wire (pts (xy 337.82 153.035) (xy 342.265 153.035))
     (stroke (width 0) (type default))
   )
+  (wire (pts (xy 297.18 29.21) (xy 277.495 29.21))
+    (stroke (width 0) (type default))
+  )
   (wire (pts (xy 297.18 136.525) (xy 305.435 136.525))
     (stroke (width 0) (type default))
   )
+  (wire (pts (xy 297.815 66.675) (xy 276.86 66.675))
+    (stroke (width 0) (type default))
+  )
   (wire (pts (xy 297.18 152.4) (xy 305.435 152.4))
     (stroke (width 0) (type default))
@@
     (stroke (width 0) (type default))
   )
-  (wire (pts (xy 333.375 50.165) (xy 356.87 50.165))
+  (wire (pts (xy 333.375 50.165) (xy 341.63 50.165))
     (stroke (width 0) (type default))
   )
@@
     (stroke (width 0) (type default))
   )
+  (wire (pts (xy 338.455 46.355) (xy 356.87 46.355))
+    (stroke (width 0) (type default))
+  )
   (wire (pts (xy 304.8 23.495) (xy 335.28 23.495))
     (stroke (width 0) (type default))
@@
     (stroke (width 0) (type default))
   )
+  (wire (pts (xy 338.455 29.21) (xy 338.455 46.355))
+    (stroke (width 0) (type default))
+  )
   (wire (pts (xy 337.82 149.86) (xy 342.265 149.86))
     (stroke (width 0) (type default))
   )
+  (wire (pts (xy 150.495 70.485) (xy 150.495 73.66))
+    (stroke (width 0) (type default))
+  )
   (wire (pts (xy 335.28 42.545) (xy 356.87 42.545))
     (stroke (width 0) (type default))
   )
+  (wire (pts (xy 305.435 66.675) (xy 341.63 66.675))
+    (stroke (width 0) (type default))
+  )
   (wire (pts (xy 262.89 55.88) (xy 276.86 55.88))
     (stroke (width 0) (type default))
@@
     (stroke (width 0) (type default))
   )
-  (wire (pts (xy 329.565 46.355) (xy 356.87 46.355))
+  (wire (pts (xy 329.565 46.355) (xy 338.455 46.355))
+    (stroke (width 0) (type default))
+  )
+  (wire (pts (xy 277.495 48.895) (xy 291.465 48.895))
     (stroke (width 0) (type default))
   )
@@
     (stroke (width 0) (type default))
   )
+  (wire (pts (xy 276.86 66.675) (xy 276.86 71.755))
+    (stroke (width 0) (type default))
+  )
   (wire (pts (xy 337.185 95.885) (xy 337.185 53.975))
     (stroke (width 0) (type default))
   )
+  (wire (pts (xy 158.115 73.025) (xy 158.115 70.485))
+    (stroke (width 0) (type default))
+  )
   (wire (pts (xy 285.75 83.82) (xy 292.1 83.82))
     (stroke (width 0) (type default))
@@
     (stroke (width 0) (type default))
   )
+  (wire (pts (xy 304.8 29.21) (xy 338.455 29.21))
+    (stroke (width 0) (type default))
+  )
+  (wire (pts (xy 151.765 70.485) (xy 150.495 70.485))
+    (stroke (width 0) (type default))
+  )
   (wire (pts (xy 276.86 71.755) (xy 298.45 71.755))
     (stroke (width 0) (type default))
@@
   )
   (wire (pts (xy 335.28 23.495) (xy 335.28 42.545))
+    (stroke (width 0) (type default))
+  )
+  (wire (pts (xy 158.115 70.485) (xy 156.845 70.485))
     (stroke (width 0) (type default))
   )
@@
     (effects (font (size 1.27 1.27)) (justify left bottom))
   )
-  (text "R85 and R86 provided for route around \ndebug of audio path as required"
-    (at 339.0003 29.739 0)
+  (text "R85 routes input 1 -> A\nR88 routes input 1 -> B\nR87 routes input 2 -> C\nR86 routes input 2 -> D"
+    (at 345.44 70.485 0)
     (effects (font (size 1.27 1.27)) (justify left bottom))
   )
@@
   (label "SDA1" (at 342.265 142.875 0) (fields_autoplaced)
     (effects (font (size 1.27 1.27)) (justify left bottom))
+  )
+  (symbol (lib_id "power:GND") (at 158.115 73.025 0) (unit 1)
+    (in_bom yes) (on_board yes) (dnp no) (fields_autoplaced)
+    (property "Reference" "#PWR094" (at 158.115 79.375 0)
+      (effects (font (size 1.27 1.27)) hide)
+    )
+    (property "Value" "GND" (at 158.115 77.47 0)
+      (effects (font (size 1.27 1.27)))
+    )
+    (property "Footprint" "" (at 158.115 73.025 0)
+      (effects (font (size 1.27 1.27)) hide)
+    )
+    (property "Datasheet" "" (at 158.115 73.025 0)
+      (effects (font (size 1.27 1.27)) hide)
+    )
+    (pin "1")
+    (instances
+      (project "Quad Joystick Mixer"
+        (path "/e9da4955-68c1-4335-ab8e-8a9cc0328d2d"
+          (reference "#PWR094") (unit 1)
+        )
+      )
+    )
   )
   (symbol (lib_id "power:+5V") (at 187.96 39.37 0) (unit 1)
@@
     )
   )
+  (symbol (lib_id "power:Earth") (at 150.495 73.66 0) (unit 1)
+    (in_bom yes) (on_board yes) (dnp no) (fields_autoplaced)
+    (property "Reference" "#PWR095" (at 150.495 80.01 0)
+      (effects (font (size 1.27 1.27)) hide)
+    )
+    (property "Value" "Earth" (at 150.495 77.47 0)
+      (effects (font (size 1.27 1.27)) hide)
+    )
+    (property "Footprint" "" (at 150.495 73.66 0)
+      (effects (font (size 1.27 1.27)) hide)
+    )
+    (property "Datasheet" "~" (at 150.495 73.66 0)
+      (effects (font (size 1.27 1.27)) hide)
+    )
+    (pin "1")
+    (instances
+      (project "Quad Joystick Mixer"
+        (path "/e9da4955-68c1-4335-ab8e-8a9cc0328d2d"
+          (reference "#PWR095") (unit 1)
+        )
+      )
+    )
+  )
   (symbol (lib_id "Device:R_US") (at 302.26 71.755 90) (unit 1)
     (in_bom yes) (on_board yes) (dnp no)
@@
     )
   )
+  (symbol (lib_id "Device:R_US") (at 301.625 66.675 90) (unit 1)
+    (in_bom yes) (on_board yes) (dnp no)
+    (property "Reference" "R87" (at 297.815 64.77 90)
+      (effects (font (size 1.27 1.27)))
+    )
+    (property "Value" "DNA" (at 305.435 64.77 90)
+      (effects (font (size 1.27 1.27)))
+    )
+    (property "Footprint" "" (at 301.879 65.659 90)
+      (effects (font (size 1.27 1.27)) hide)
+    )
+    (property "Datasheet" "~" (at 301.625 66.675 0)
+      (effects (font (size 1.27 1.27)) hide)
+    )
+    (pin "1")
+    (pin "2")
+    (instances
+      (project "Quad Joystick Mixer"
+        (path "/e9da4955-68c1-4335-ab8e-8a9cc0328d2d"
+          (reference "R87") (unit 1)
+        )
+      )
+    )
+  )
+  (symbol (lib_id "Device:NetTie_2") (at 154.305 70.485 0) (unit 1)
+    (in_bom no) (on_board yes) (dnp no) (fields_autoplaced)
+    (property "Reference" "NT1" (at 154.305 66.04 0)
+      (effects (font (size 1.27 1.27)))
+    )
+    (property "Value" "NetTie_2" (at 154.305 68.58 0)
+      (effects (font (size 1.27 1.27)))
+    )
+    (property "Footprint" "NetTie:NetTie-2_SMD_Pad2.0mm" (at 154.305 70.485 0)
+      (effects (font (size 1.27 1.27)) hide)
+    )
+    (property "Datasheet" "~" (at 154.305 70.485 0)
+      (effects (font (size 1.27 1.27)) hide)
+    )
+    (pin "1")
+    (pin "2")
+    (instances
+      (project "Quad Joystick Mixer"
+        (path "/e9da4955-68c1-4335-ab8e-8a9cc0328d2d"
+          (reference "NT1") (unit 1)
+        )
+      )
+    )
+  )
   (symbol (lib_id "Device:R_US") (at 300.99 23.495 90) (unit 1)
     (in_bom yes) (on_board yes) (dnp no)
@@
         )
       )
+    )
+  )
+  (symbol (lib_id "Device:R_US") (at 300.99 29.21 90) (unit 1)
+    (in_bom yes) (on_board yes) (dnp no)
+    (property "Reference" "R88" (at 297.18 27.305 90)
+      (effects (font (size 1.27 1.27)))
+    )
+    (property "Value" "DNA" (at 304.8 27.305 90)
+      (effects (font (size 1.27 1.27)))
+    )
+    (property "Footprint" "" (at 301.244 28.194 90)
+      (effects (font (size 1.27 1.27)) hide)
+    )
+    (property "Datasheet" "~" (at 300.99 29.21 0)
+      (effects (font (size 1.27 1.27)) hide)
+    )
+    (pin "1")
+    (pin "2")
+    (instances
+      (project "Quad Joystick Mixer"
+        (path "/e9da4955-68c1-4335-ab8e-8a9cc0328d2d"
+          (reference "R88") (unit 1)
+        )
+      )
