File: Quad Joystick Mixer/userInterface.kicad_sch (KiCad schematic)
At the start: 23 parts, among them SW2 Stompbox 1P8T Rotary, U4 OPA1692xD

Commit message: finished first draft of the schematic
Parts:
- added C13 (x3): 0.1uF, Capacitor_SMD:C_0805_2012Metric_Pad1.18x1.45mm_HandSolder, symbol Device:C
- added D22, D23, D24: SMAJ3.3A, Diode_SMD:D_SMA, symbol Diode:SMAJ5.0A
- added D8 (x2): LED, LED_THT:LED_D3.0mm_FlatTop, symbol Device:LED
- added Q1, Q2: 2N7002, Package_TO_SOT_SMD:SOT-23, symbol Transistor_FET:2N7002
- added R78, R80: 200, symbol Device:R_US
- added R79, R81, R82, R83, R84: 10k, symbol Device:R_US
- added SW3, SW4, SW5: Cherry MX, Button_Switch_Keyboard:SW_Cherry_MX_1.00u_PCB, symbol Switch:SW_SPST
Connections:
- net +3.3V: now also D8.2 (A), D8.2 (A), R82.2, R83.2, R84.2
- net Earth: now also C13.2, C13.2, C13.2, D22.2 (A2), D23.2 (A2), D24.2 (A2), Q1.2 (S), Q2.2 (S), R79.1, R81.1, SW3.2 (B), SW4.2 (B), SW5.2 (B)
- new net: D8.1 (K), R78.2
- new net: Q1.3 (D), R78.1
- new net: D8.1 (K), R80.2
- new net: Q2.3 (D), R80.1
- new net Button_1: C13.1, D22.1 (A1), R82.1, SW3.1 (A)
- new net Button_2: C13.1, D23.1 (A1), R83.1, SW4.1 (A)
- new net Button_3: C13.1, D24.1 (A1), R84.1, SW5.1 (A)
- new net LED_1: Q1.1 (G), R79.2
- new net LED_2: Q2.1 (G), R81.2
Other:
- note added: "User Interface Ins and Outs"
- title: (none) -> Quadrophonic Joystick Mixer

Commit message: ok the draft wasn't done but now i think it is
Parts:
- added TP1 (x3): TestPoint, TestPoint:TestPoint_THTPad_D1.5mm_Drill0.7mm, symbol Connector:TestPoint
Connections:
- net AB_control: now also TP1.1
- net CD_control: now also TP1.1
- net Channel Selection: now also TP1.1
Changed lines of the file:
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@@
   (junction (at 377.825 60.96) (diameter 0) (color 0 0 0 0)
   )
+  (junction (at 332.105 80.645) (diameter 0) (color 0 0 0 0)
+  )
   (junction (at 116.84 54.61) (diameter 0) (color 0 0 0 0)
   )
@@
   (junction (at 73.025 158.115) (diameter 0) (color 0 0 0 0)
   )
+  (junction (at 125.095 54.61) (diameter 0) (color 0 0 0 0)
+  )
   (junction (at 328.93 80.645) (diameter 0) (color 0 0 0 0)
   )
+  (junction (at 125.095 90.17) (diameter 0) (color 0 0 0 0)
+  )
   (junction (at 332.74 153.035) (diameter 0) (color 0 0 0 0)
   )
@@
   )
   (no_connect (at 360.68 76.2))
-  (wire (pts (xy 122.555 90.17) (xy 127 90.17))
+  (wire (pts (xy 125.095 50.165) (xy 125.095 54.61))
+    (stroke (width 0) (type default))
+  )
+  (wire (pts (xy 122.555 90.17) (xy 125.095 90.17))
     (stroke (width 0) (type default))
   )
@@
     (stroke (width 0) (type default))
   )
+  (wire (pts (xy 125.095 54.61) (xy 127 54.61))
+    (stroke (width 0) (type default))
+  )
   (wire (pts (xy 253.365 156.845) (xy 253.365 153.035))
     (stroke (width 0) (type default))
@@
     (stroke (width 0) (type default))
   )
+  (wire (pts (xy 125.095 90.17) (xy 127 90.17))
+    (stroke (width 0) (type default))
+  )
   (wire (pts (xy 108.585 169.545) (xy 108.585 171.45))
     (stroke (width 0) (type default))
@@
     (stroke (width 0) (type default))
   )
+  (wire (pts (xy 126.365 50.165) (xy 125.095 50.165))
+    (stroke (width 0) (type default))
+  )
   (wire (pts (xy 118.745 98.425) (xy 95.885 98.425))
     (stroke (width 0) (type default))
@@
     (stroke (width 0) (type default))
   )
-  (wire (pts (xy 328.93 80.645) (xy 334.645 80.645))
+  (wire (pts (xy 328.93 80.645) (xy 332.105 80.645))
     (stroke (width 0) (type default))
   )
@@
     (stroke (width 0) (type default))
   )
-  (wire (pts (xy 121.92 54.61) (xy 127 54.61))
+  (wire (pts (xy 121.92 54.61) (xy 125.095 54.61))
     (stroke (width 0) (type default))
   )
@@
     (stroke (width 0) (type default))
   )
+  (wire (pts (xy 332.105 80.645) (xy 334.645 80.645))
+    (stroke (width 0) (type default))
+  )
   (wire (pts (xy 266.065 165.735) (xy 266.065 167.64))
     (stroke (width 0) (type default))
@@
     (stroke (width 0) (type default))
   )
+  (wire (pts (xy 127 85.725) (xy 125.095 85.725))
+    (stroke (width 0) (type default))
+  )
   (wire (pts (xy 377.825 60.96) (xy 377.825 63.5))
     (stroke (width 0) (type default))
@@
     (stroke (width 0) (type default))
   )
+  (wire (pts (xy 334.01 76.835) (xy 332.105 76.835))
+    (stroke (width 0) (type default))
+  )
   (wire (pts (xy 60.96 55.88) (xy 60.96 57.785))
     (stroke (width 0) (type default))
@@
     (stroke (width 0) (type default))
   )
+  (wire (pts (xy 125.095 85.725) (xy 125.095 90.17))
+    (stroke (width 0) (type default))
+  )
   (wire (pts (xy 73.025 158.115) (xy 69.85 158.115))
     (stroke (width 0) (type default))
@@
   )
   (wire (pts (xy 332.74 153.035) (xy 332.74 156.21))
+    (stroke (width 0) (type default))
+  )
+  (wire (pts (xy 332.105 76.835) (xy 332.105 80.645))
     (stroke (width 0) (type default))
   )
@@
     (effects (font (size 1.27 1.27)) (justify left))
   )
+  (symbol (lib_id "Connector:TestPoint") (at 127 85.725 270) (unit 1)
+    (in_bom yes) (on_board yes) (dnp no) (fields_autoplaced)
+    (property "Reference" "TP1" (at 132.715 85.725 90)
+      (effects (font (size 1.27 1.27)) (justify left))
+    )
+    (property "Value" "TestPoint" (at 129.032 87.63 0)
+      (effects (font (size 1.27 1.27)) (justify left) hide)
+    )
+    (property "Footprint" "TestPoint:TestPoint_THTPad_D1.5mm_Drill0.7mm" (at 127 90.805 0)
+      (effects (font (size 1.27 1.27)) hide)
+    )
+    (property "Datasheet" "~" (at 127 90.805 0)
+      (effects (font (size 1.27 1.27)) hide)
+    )
+    (pin "1")
+    (instances
+      (project "Quad Joystick Mixer"
+        (path "/e9da4955-68c1-4335-ab8e-8a9cc0328d2d/70e873e8-c2f7-42de-91d7-3f147d0d972e"
+          (reference "TP1") (unit 1)
+        )
+        (path "/e9da4955-68c1-4335-ab8e-8a9cc0328d2d/2bfe18f6-ab55-4efd-b5e1-a61472c26ad3"
+          (reference "TP21") (unit 1)
+        )
+      )
+    )
+  )
   (symbol (lib_id "Device:C") (at 253.365 160.655 0) (unit 1)
     (in_bom yes) (on_board yes) (dnp no) (fields_autoplaced)
@@
         (path "/e9da4955-68c1-4335-ab8e-8a9cc0328d2d/2bfe18f6-ab55-4efd-b5e1-a61472c26ad3"
           (reference "R72") (unit 1)
+        )
+      )
+    )
+  )
+  (symbol (lib_id "Connector:TestPoint") (at 126.365 50.165 270) (unit 1)
+    (in_bom yes) (on_board yes) (dnp no) (fields_autoplaced)
+    (property "Reference" "TP1" (at 132.08 50.165 90)
+      (effects (font (size 1.27 1.27)) (justify left))
+    )
+    (property "Value" "TestPoint" (at 128.397 52.07 0)
+      (effects (font (size 1.27 1.27)) (justify left) hide)
+    )
+    (property "Footprint" "TestPoint:TestPoint_THTPad_D1.5mm_Drill0.7mm" (at 126.365 55.245 0)
+      (effects (font (size 1.27 1.27)) hide)
+    )
+    (property "Datasheet" "~" (at 126.365 55.245 0)
+      (effects (font (size 1.27 1.27)) hide)
+    )
+    (pin "1")
+    (instances
+      (project "Quad Joystick Mixer"
+        (path "/e9da4955-68c1-4335-ab8e-8a9cc0328d2d/70e873e8-c2f7-42de-91d7-3f147d0d972e"
+          (reference "TP1") (unit 1)
+        )
+        (path "/e9da4955-68c1-4335-ab8e-8a9cc0328d2d/2bfe18f6-ab55-4efd-b5e1-a61472c26ad3"
+          (reference "TP20") (unit 1)
         )
       )
@@
         )
       )
+    )
+  )
+  (symbol (lib_id "Connector:TestPoint") (at 334.01 76.835 270) (unit 1)
+    (in_bom yes) (on_board yes) (dnp no) (fields_autoplaced)
+    (property "Reference" "TP1" (at 339.725 76.835 90)
+      (effects (font (size 1.27 1.27)) (justify left))
+    )
+    (property "Value" "TestPoint" (at 336.042 78.74 0)
+      (effects (font (size 1.27 1.27)) (justify left) hide)
+    )
+    (property "Footprint" "TestPoint:TestPoint_THTPad_D1.5mm_Drill0.7mm" (at 334.01 81.915 0)
+      (effects (font (size 1.27 1.27)) hide)
+    )
+    (property "Datasheet" "~" (at 334.01 81.915 0)
+      (effects (font (size 1.27 1.27)) hide)
+    )
+    (pin "1")
+    (instances
+      (project "Quad Joystick Mixer"
+        (path "/e9da4955-68c1-4335-ab8e-8a9cc0328d2d/70e873e8-c2f7-42de-91d7-3f147d0d972e"
+          (reference "TP1") (unit 1)
+        )
+        (path "/e9da4955-68c1-4335-ab8e-8a9cc0328d2d/2bfe18f6-ab55-4efd-b5e1-a61472c26ad3"
+          (reference "TP22") (unit 1)
+        )
+      )

Commit message: clean up after review, working through BOM
Parts:
- D18, D19: footprint (none) -> Diode_SMD:D_SOD-123; DK PN (none) -> DDZ9684-7DICT-ND; MPN (none) -> DDZ9684-7
- D22, D23, D24: value SMAJ3.3A -> SMAJ5.0A; DK PN (none) -> SMAJ5.0A-FDICT-ND; MPN (none) -> SMAJ5.0A-13-F
- Q1, Q2: DK PN (none) -> 2N7002-TPMSCT-ND; MPN (none) -> 2N7002-TP
Changed lines of the file:
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@@
       (effects (font (size 1.27 1.27)) (justify left))
     )
-    (property "Footprint" "" (at 121.92 66.04 0)
+    (property "Footprint" "Diode_SMD:D_SOD-123" (at 121.92 66.04 0)
       (effects (font (size 1.27 1.27)) hide)
     )
     (property "Datasheet" "~" (at 121.92 66.04 0)
+      (effects (font (size 1.27 1.27)) hide)
+    )
+    (property "DK PN" "DDZ9684-7DICT-ND" (at 121.92 66.04 0)
+      (effects (font (size 1.27 1.27)) hide)
+    )
+    (property "MPN" "DDZ9684-7" (at 121.92 66.04 0)
       (effects (font (size 1.27 1.27)) hide)
     )
@@
       (effects (font (size 1.27 1.27)) (justify left))
     )
-    (property "Value" "SMAJ3.3A" (at 319.405 163.195 90)
+    (property "Value" "SMAJ5.0A" (at 319.405 163.195 90)
       (effects (font (size 1.27 1.27)) (justify left))
     )
@@
     )
     (property "Datasheet" "https://www.littelfuse.com/media?resourcetype=datasheets&itemid=75e32973-b177-4ee3-a0ff-cedaf1abdb93&filename=smaj-datasheet" (at 316.865 160.655 0)
+      (effects (font (size 1.27 1.27)) hide)
+    )
+    (property "DK PN" "SMAJ5.0A-FDICT-ND" (at 316.865 161.925 0)
+      (effects (font (size 1.27 1.27)) hide)
+    )
+    (property "MPN" "SMAJ5.0A-13-F" (at 316.865 161.925 0)
       (effects (font (size 1.27 1.27)) hide)
     )
@@
       (effects (font (size 1.27 1.27)) (justify left) hide)
     )
+    (property "DK PN" "2N7002-TPMSCT-ND" (at 64.77 158.115 0)
+      (effects (font (size 1.27 1.27)) hide)
+    )
+    (property "MPN" "2N7002-TP" (at 64.77 158.115 0)
+      (effects (font (size 1.27 1.27)) hide)
+    )
     (pin "1")
     (pin "2")
@@
       (effects (font (size 1.27 1.27)) (justify left))
     )
-    (property "Value" "SMAJ3.3A" (at 217.17 163.83 90)
+    (property "Value" "SMAJ5.0A" (at 217.17 163.83 90)
       (effects (font (size 1.27 1.27)) (justify left))
     )
@@
     )
     (property "Datasheet" "https://www.littelfuse.com/media?resourcetype=datasheets&itemid=75e32973-b177-4ee3-a0ff-cedaf1abdb93&filename=smaj-datasheet" (at 214.63 161.29 0)
+      (effects (font (size 1.27 1.27)) hide)
+    )
+    (property "DK PN" "SMAJ5.0A-FDICT-ND" (at 214.63 162.56 0)
+      (effects (font (size 1.27 1.27)) hide)
+    )
+    (property "MPN" "SMAJ5.0A-13-F" (at 214.63 162.56 0)
       (effects (font (size 1.27 1.27)) hide)
     )
@@
       (effects (font (size 1.27 1.27)) (justify left))
     )
-    (property "Footprint" "" (at 122.555 101.6 0)
+    (property "Footprint" "Diode_SMD:D_SOD-123" (at 122.555 101.6 0)
       (effects (font (size 1.27 1.27)) hide)
     )
     (property "Datasheet" "~" (at 122.555 101.6 0)
+      (effects (font (size 1.27 1.27)) hide)
+    )
+    (property "DK PN" "DDZ9684-7DICT-ND" (at 122.555 101.6 0)
+      (effects (font (size 1.27 1.27)) hide)
+    )
+    (property "MPN" "DDZ9684-7" (at 122.555 101.6 0)
       (effects (font (size 1.27 1.27)) hide)
     )
@@
       (effects (font (size 1.27 1.27)) (justify left) hide)
     )
+    (property "DK PN" "2N7002-TPMSCT-ND" (at 100.33 158.75 0)
+      (effects (font (size 1.27 1.27)) hide)
+    )
+    (property "MPN" "2N7002-TP" (at 100.33 158.75 0)
+      (effects (font (size 1.27 1.27)) hide)
+    )
     (pin "1")
     (pin "2")
@@
       (effects (font (size 1.27 1.27)) (justify left))
     )
-    (property "Value" "SMAJ3.3A" (at 268.605 163.195 90)
+    (property "Value" "SMAJ5.0A" (at 268.605 163.195 90)
       (effects (font (size 1.27 1.27)) (justify left))
     )
@@
       (effects (font (size 1.27 1.27)) hide)
     )
+    (property "DK PN" "SMAJ5.0A-FDICT-ND" (at 266.065 161.925 0)
+      (effects (font (size 1.27 1.27)) hide)
+    )
+    (property "MPN" "SMAJ5.0A-13-F" (at 266.065 161.925 0)
+      (effects (font (size 1.27 1.27)) hide)
+    )

Commit message: finish adding parts to the BOM
Parts:
- C13, C5, D18, D19, D22, D23, D24, Q1, Q2: Source (none) -> DK
- D8, SW2: Source (none) -> SBP
- R62: footprint (none) -> Resistor_SMD:R_0805_2012Metric_Pad1.20x1.40mm_HandSolder; DK PN (none) -> 311-1.43KCRCT-ND; MPN (none) -> RC0805FR-071K43L; Source (none) -> DK
- R63: footprint (none) -> Resistor_SMD:R_0805_2012Metric_Pad1.20x1.40mm_HandSolder; DK PN (none) -> RMCF0805FT3K32CT-ND; MPN (none) -> RMCF0805FT3K32; Source (none) -> DK
- R64, R65: footprint (none) -> Resistor_SMD:R_0805_2012Metric_Pad1.20x1.40mm_HandSolder; DK PN (none) -> 311-100CRCT-ND; MPN (none) -> RC0805FR-07100RL; Source (none) -> DK
- R72: footprint (none) -> Resistor_SMD:R_0805_2012Metric_Pad1.20x1.40mm_HandSolder; DK PN (none) -> RMCF0805FT6K04CT-ND; MPN (none) -> RMCF0805FT6K04; Source (none) -> DK
- R73, R77, R79, R81, R82, R83, R84: footprint (none) -> Resistor_SMD:R_0805_2012Metric_Pad1.20x1.40mm_HandSolder; DK PN (none) -> RMCF0805JT10K0CT-ND; MPN (none) -> RMCF0805JT10K0; Source (none) -> DK
- R74: footprint (none) -> Resistor_SMD:R_0805_2012Metric_Pad1.20x1.40mm_HandSolder; DK PN (none) -> RMCF0805FT16K5CT-ND; MPN (none) -> RMCF0805FT16K5; Source (none) -> DK
- R75: footprint (none) -> Resistor_SMD:R_0805_2012Metric_Pad1.20x1.40mm_HandSolder; DK PN (none) -> RMCF0805FT30K1CT-ND; MPN (none) -> RMCF0805FT30K1; Source (none) -> DK
- R76: footprint (none) -> Resistor_SMD:R_0805_2012Metric_Pad1.20x1.40mm_HandSolder; DK PN (none) -> RMCF0805FT71K5CT-ND; MPN (none) -> RMCF0805FT71K5; Source (none) -> DK
- R78, R80: footprint (none) -> Resistor_SMD:R_0805_2012Metric_Pad1.20x1.40mm_HandSolder; DK PN (none) -> RMCF0805FT200RCT-ND; MPN (none) -> RMCF0805FT200R; Source (none) -> DK
- RV3, RV4: MPN (none) -> Joystick; Source (none) -> SBP
- SW3, SW4, SW5: DK PN (none) -> CH160-ND; MPN (none) -> MX1A-11NW; Source (none) -> DK
- TP1: Source (none) -> NA
- U4: value OPA1692xD -> TL072; DK PN (none) -> 296-TL072HIDRCT-ND; MPN (none) -> TL072HIDR; Source (none) -> DK

Commit message: work through DRC errors
Parts:
- added J8, J9: XH-A, Connector_JST:JST_XH_B3B-XH-AM_1x03_P2.50mm_Vertical, symbol Connector:Conn_01x03_Pin
Connections:
- net +3.3V: now also J8.1 (Pin_1), J9.1 (Pin_1)
- net Earth: now also J8.3 (Pin_3), J9.3 (Pin_3)
- net at R64.1, RV3.2: now also J8.2 (Pin_2)
- net at R65.1, RV4.2: now also J9.2 (Pin_2)
Other:
- moved on the sheet: C13

Commit message: changed power supply design and everything re routed
Parts:
- J8, J9: Source (none) -> SBP
Changed lines of the file:
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@@
+      (effects (font (size 1.27 1.27)) hide)
+    )
+    (property "Source" "SBP" (at 41.91 52.705 0)
       (effects (font (size 1.27 1.27)) hide)
     )
@@
       (effects (font (size 1.27 1.27)) hide)
     )
+    (property "Source" "SBP" (at 45.085 91.44 0)
+      (effects (font (size 1.27 1.27)) hide)
+    )
