File: Hardware/Quad Joystick Mixer/Quad Joystick Mixer.kicad_pcb (KiCad board)
At the start: 4 copper layers, 189.3 x 134.8 mm, 228 parts, among them J1 XH-B4B-XH, J2 NMJ6HCD, J3 NMJ6HCD, J4 NMJ6HCD, J5 NMJ6HCD, J6 NMJ6HCD, J7 NMJ6HCD, J8 XH-A, J9 XH-A, Q1 2N7002, Q2 2N7002, SW2 Stompbox 1P8T Rotary, SW3 Cherry MX, SW4 Cherry MX, SW5 Cherry MX, SW6 Cherry MX, SW7 Cherry MX, U1 L78M12ACDT-TR, U10 TL072, U11 TL072, U12 TL072, U13 DS1881Z-050+, U14 TL072, U16 TL072, U17 DS1881Z-050+, U19 TL072, U2 MC79L12ABDG, U20 Teensy4.0, U4 TL072, U5 MCP1755T-5002E/OT, U6 TL072, U7 TL072, U8 DS1881Z-050+, U9 DS1881Z-050+

Commit message: add FW, updated README
Parts:
- added REF**: MountingHole_2.7mm_M2.5, MountingHole:MountingHole_2.7mm_M2.5, F.Cu at (243.2, 32.8)
- added REF**: MountingHole_2.7mm_M2.5, MountingHole:MountingHole_2.7mm_M2.5, F.Cu at (60.4, 161.0)
- added REF**: MountingHole_2.7mm_M2.5, MountingHole:MountingHole_2.7mm_M2.5, F.Cu at (138.8, 74.0)
- added REF**: MountingHole_2.7mm_M2.5, MountingHole:MountingHole_2.7mm_M2.5, F.Cu at (124.0, 127.0)
- added REF**: MountingHole_2.7mm_M2.5, MountingHole:MountingHole_2.7mm_M2.5, F.Cu at (181.4, 161.0)
- added REF**: MountingHole_2.7mm_M2.5, MountingHole:MountingHole_2.7mm_M2.5, F.Cu at (236.2, 112.8)
- added REF**: MountingHole_2.7mm_M2.5, MountingHole:MountingHole_2.7mm_M2.5, F.Cu at (60.4, 32.8)
- added REF**: MountingHole_2.7mm_M2.5, MountingHole:MountingHole_2.7mm_M2.5, F.Cu at (139.0, 32.8)
- added REF**: MountingHole_2.7mm_M2.5, MountingHole:MountingHole_2.7mm_M2.5, F.Cu at (243.2, 161.0)
- added REF**: MountingHole_2.7mm_M2.5, MountingHole:MountingHole_2.7mm_M2.5, F.Cu at (76.6, 101.4)
Routing:
- net /Teensy/Button_3: track 129.2 -> 133.1 mm
- net /Audio Output/D: track 220.5 -> 219.5 mm
- net +3.3V: track 259.3 -> 258.5 mm, vias 8 -> 11
- net +12V: track 78.2 -> 77.5 mm
- net Earth: track 100.4 -> 99.9 mm
Other:
- board text added: "03/08/24 BOARD VERSION"
- board text added: "A Out"
- board text added: "B Out"
- board text added: "Button 1"
- board text added: "Button 2"
- board text added: "Button 3"
- board text added: "C Out"
- board text added: "Channel Select"
- board text added: "D Out"
- board text added: "Digital Pots for Channel 1"
- board text added: "Digital Pots for Channel 2"
- board text added: "Input 1"
- board text added: "Input 1 Gain"
- board text added: "Input 2"
- board text added: "Input 2 Gain"
- board text added: "Joystick Connections - Pots placed for development use"
- board text added: "QUAD JOYSTICK MIXER V1"
- board text added: "Teensy PROG"
- board text added: "Teensy Power"
- board text added: "To Meanwell RT-50C"

Commit message: add mechanical integration stuff
Parts:
- added REF**: Meanwell RT-50C, Eyewool Mechanicals:Meanwell RT-50C, F.Cu at (148.6, 105.2)
- moved C26 151.9 mm to (360.1, 162.1)
- moved C29 151.9 mm to (368.6, 164.6)
- moved C30 151.9 mm to (364.1, 164.6)
- moved C31 151.9 mm to (368.1, 155.6)
- moved C35 151.9 mm to (330.9, 119.0)
- moved C38 151.9 mm to (330.9, 116.5)
- moved C40 151.9 mm to (304.8, 117.8)
- moved C46 151.9 mm to (334.4, 111.3)
- moved C55 151.9 mm to (371.3, 146.5)
- moved C65 151.9 mm to (349.8, 107.8)
- moved C66 151.9 mm to (362.3, 109.3)
- moved C67 151.9 mm to (387.5, 106.6)
- moved C68 151.9 mm to (362.3, 106.3)
- moved C69 151.9 mm to (378.5, 114.6)
- moved C70 151.9 mm to (353.8, 113.3)
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Other:
- board text added: "3.819 in. x 3.898 in."
- board text added: "ORIGIN"
- board text added: "POWER SUPPLY"
